Commit message: can move joints

File: naranjelio.urdf.xacro (robot description, xacro)
@@ -4,5 +4,5 @@
 <!-- |    EDITING THIS FILE BY HAND IS NOT RECOMMENDED                                 | -->
 <!-- =================================================================================== -->
-<robot name="naranjelio">
+<robot name="naranjelio" xmlns:xacro="http://www.ros.org/wiki/xacro">
   <material name="silver">
     <color rgba="0.700 0.700 0.700 1.000" />
@@ -128,84 +128,87 @@
     </actuator>
   </transmission>
-  <transmission name="Revolute 45_tran">
-    <type>transmission_interface/SimpleTransmission</type>
-    <joint name="Revolute 45">
-      <hardwareInterface>hardware_interface/EffortJointInterface</hardwareInterface>
-    </joint>
-    <actuator name="Revolute 45_actr">
-      <hardwareInterface>hardware_interface/EffortJointInterface</hardwareInterface>
-      <mechanicalReduction>1</mechanicalReduction>
-    </actuator>
-  </transmission>
-  <transmission name="Revolute 46_tran">
-    <type>transmission_interface/SimpleTransmission</type>
-    <joint name="Revolute 46">
-      <hardwareInterface>hardware_interface/EffortJointInterface</hardwareInterface>
-    </joint>
-    <actuator name="Revolute 46_actr">
-      <hardwareInterface>hardware_interface/EffortJointInterface</hardwareInterface>
-      <mechanicalReduction>1</mechanicalReduction>
-    </actuator>
-  </transmission>
-  <transmission name="Revolute 47_tran">
-    <type>transmission_interface/SimpleTransmission</type>
-    <joint name="Revolute 47">
-      <hardwareInterface>hardware_interface/EffortJointInterface</hardwareInterface>
-    </joint>
-    <actuator name="Revolute 47_actr">
-      <hardwareInterface>hardware_interface/EffortJointInterface</hardwareInterface>
-      <mechanicalReduction>1</mechanicalReduction>
-    </actuator>
-  </transmission>
-  <transmission name="Revolute 48_tran">
-    <type>transmission_interface/SimpleTransmission</type>
-    <joint name="Revolute 48">
-      <hardwareInterface>hardware_interface/EffortJointInterface</hardwareInterface>
-    </joint>
-    <actuator name="Revolute 48_actr">
-      <hardwareInterface>hardware_interface/EffortJointInterface</hardwareInterface>
-      <mechanicalReduction>1</mechanicalReduction>
-    </actuator>
-  </transmission>
-  <transmission name="Revolute 49_tran">
-    <type>transmission_interface/SimpleTransmission</type>
-    <joint name="Revolute 49">
-      <hardwareInterface>hardware_interface/EffortJointInterface</hardwareInterface>
-    </joint>
-    <actuator name="Revolute 49_actr">
-      <hardwareInterface>hardware_interface/EffortJointInterface</hardwareInterface>
-      <mechanicalReduction>1</mechanicalReduction>
-    </actuator>
-  </transmission>
-  <transmission name="Revolute 50_tran">
-    <type>transmission_interface/SimpleTransmission</type>
-    <joint name="Revolute 50">
-      <hardwareInterface>hardware_interface/EffortJointInterface</hardwareInterface>
-    </joint>
-    <actuator name="Revolute 50_actr">
-      <hardwareInterface>hardware_interface/EffortJointInterface</hardwareInterface>
-      <mechanicalReduction>1</mechanicalReduction>
-    </actuator>
-  </transmission>
-  <transmission name="Revolute 51_tran">
-    <type>transmission_interface/SimpleTransmission</type>
-    <joint name="Revolute 51">
-      <hardwareInterface>hardware_interface/EffortJointInterface</hardwareInterface>
-    </joint>
-    <actuator name="Revolute 51_actr">
-      <hardwareInterface>hardware_interface/EffortJointInterface</hardwareInterface>
-      <mechanicalReduction>1</mechanicalReduction>
-    </actuator>
-  </transmission>
-  <transmission name="Revolute 52_tran">
-    <type>transmission_interface/SimpleTransmission</type>
-    <joint name="Revolute 52">
-      <hardwareInterface>hardware_interface/EffortJointInterface</hardwareInterface>
-    </joint>
-    <actuator name="Revolute 52_actr">
-      <hardwareInterface>hardware_interface/EffortJointInterface</hardwareInterface>
-      <mechanicalReduction>1</mechanicalReduction>
-    </actuator>
-  </transmission>
+  <transmission name="Revolute_45_tran">
+    <type>transmission_interface/SimpleTransmission</type>
+    <joint name="Revolute_45">
+      <hardwareInterface>hardware_interface/EffortJointInterface</hardwareInterface>
+    </joint>
+    <actuator name="Revolute_45_actr">
+      <hardwareInterface>hardware_interface/EffortJointInterface</hardwareInterface>
+      <mechanicalReduction>1</mechanicalReduction>
+    </actuator>
+  </transmission>
+  <transmission name="Revolute_46_tran">
+    <type>transmission_interface/SimpleTransmission</type>
+    <joint name="Revolute_46">
+      <hardwareInterface>hardware_interface/EffortJointInterface</hardwareInterface>
+    </joint>
+    <actuator name="Revolute_46_actr">
+      <hardwareInterface>hardware_interface/EffortJointInterface</hardwareInterface>
+      <mechanicalReduction>1</mechanicalReduction>
+    </actuator>
+  </transmission>
+  <transmission name="Revolute_47_tran">
+    <type>transmission_interface/SimpleTransmission</type>
+    <joint name="Revolute_47">
+      <hardwareInterface>hardware_interface/EffortJointInterface</hardwareInterface>
+    </joint>
+    <actuator name="Revolute_47_actr">
+      <hardwareInterface>hardware_interface/EffortJointInterface</hardwareInterface>
+      <mechanicalReduction>1</mechanicalReduction>
+    </actuator>
+  </transmission>
+  <transmission name="Revolute_48_tran">
+    <type>transmission_interface/SimpleTransmission</type>
+    <joint name="Revolute_48">
+      <hardwareInterface>hardware_interface/EffortJointInterface</hardwareInterface>
+    </joint>
+    <actuator name="Revolute_48_actr">
+      <hardwareInterface>hardware_interface/EffortJointInterface</hardwareInterface>
+      <mechanicalReduction>1</mechanicalReduction>
+    </actuator>
+  </transmission>
+  <transmission name="Revolute_49_tran">
+    <type>transmission_interface/SimpleTransmission</type>
+    <joint name="Revolute_49">
+      <hardwareInterface>hardware_interface/EffortJointInterface</hardwareInterface>
+    </joint>
+    <actuator name="Revolute_49_actr">
+      <hardwareInterface>hardware_interface/EffortJointInterface</hardwareInterface>
+      <mechanicalReduction>1</mechanicalReduction>
+    </actuator>
+  </transmission>
+  <transmission name="Revolute_50_tran">
+    <type>transmission_interface/SimpleTransmission</type>
+    <joint name="Revolute_50">
+      <hardwareInterface>hardware_interface/EffortJointInterface</hardwareInterface>
+    </joint>
+    <actuator name="Revolute_50_actr">
+      <hardwareInterface>hardware_interface/EffortJointInterface</hardwareInterface>
+      <mechanicalReduction>1</mechanicalReduction>
+    </actuator>
+  </transmission>
+  <transmission name="Revolute_51_tran">
+    <type>transmission_interface/SimpleTransmission</type>
+    <joint name="Revolute_51">
+      <hardwareInterface>hardware_interface/EffortJointInterface</hardwareInterface>
+    </joint>
+    <actuator name="Revolute_51_actr">
+      <hardwareInterface>hardware_interface/EffortJointInterface</hardwareInterface>
+      <mechanicalReduction>1</mechanicalReduction>
+    </actuator>
+  </transmission>
+  <transmission name="Revolute_52_tran">
+    <type>transmission_interface/SimpleTransmission</type>
+    <joint name="Revolute_52">
+      <hardwareInterface>hardware_interface/EffortJointInterface</hardwareInterface>
+    </joint>
+    <actuator name="Revolute_52_actr">
+      <hardwareInterface>hardware_interface/EffortJointInterface</hardwareInterface>
+      <mechanicalReduction>1</mechanicalReduction>
+    </actuator>
+  </transmission>
+  <plugin filename="gz-sim-joint-state-publisher-system"
+      name="gz::sim::systems::JointStatePublisher">
+    </plugin>
   <gazebo>
     <plugin filename="gz_ros2_control-system" name="gz_ros2_control::GazeboSimROS2ControlPlugin">
@@ -467,5 +470,5 @@
       <geometry>
         <mesh
-          filename="file:///home/devuser/sinfonia/Documents/repos_varios/naranjelio_ws/install/naranjelio_description/share/naranjelio_description/meshes/base_link.stl"
+          filename="file://$(env NARANJELIO_HOME)/meshes/base_link.stl"
           scale="0.001 0.001 0.001" />
       </geometry>
@@ -476,5 +479,5 @@
       <geometry>
         <mesh
-          filename="file:///home/devuser/sinfonia/Documents/repos_varios/naranjelio_ws/install/naranjelio_description/share/naranjelio_description/meshes/base_link.stl"
+          filename="file://$(env NARANJELIO_HOME)/meshes/base_link.stl"
           scale="0.001 0.001 0.001" />
       </geometry>
@@ -491,5 +494,5 @@
       <geometry>
         <mesh
-          filename="file:///home/devuser/sinfonia/Documents/repos_varios/naranjelio_ws/install/naranjelio_description/share/naranjelio_description/meshes/FrontIzq_1.stl"
+          filename="file://$(env NARANJELIO_HOME)/meshes/FrontIzq_1.stl"
           scale="0.001 0.001 0.001" />
       </geometry>
@@ -500,5 +503,5 @@
       <geometry>
         <mesh
-          filename="file:///home/devuser/sinfonia/Documents/repos_varios/naranjelio_ws/install/naranjelio_description/share/naranjelio_description/meshes/FrontIzq_1.stl"
+          filename="file://$(env NARANJELIO_HOME)/meshes/FrontIzq_1.stl"
           scale="0.001 0.001 0.001" />
       </geometry>
@@ -515,5 +518,5 @@
       <geometry>
         <mesh
-          filename="file:///home/devuser/sinfonia/Documents/repos_varios/naranjelio_ws/install/naranjelio_description/share/naranjelio_description/meshes/FrontDer_1.stl"
+          filename="file://$(env NARANJELIO_HOME)/meshes/FrontDer_1.stl"
           scale="0.001 0.001 0.001" />
       </geometry>
@@ -524,5 +527,5 @@
       <geometry>
         <mesh
-          filename="file:///home/devuser/sinfonia/Documents/repos_varios/naranjelio_ws/install/naranjelio_description/share/naranjelio_description/meshes/FrontDer_1.stl"
+          filename="file://$(env NARANJELIO_HOME)/meshes/FrontDer_1.stl"
           scale="0.001 0.001 0.001" />
       </geometry>
@@ -539,5 +542,5 @@
       <geometry>
         <mesh
-          filename="file:///home/devuser/sinfonia/Documents/repos_varios/naranjelio_ws/install/naranjelio_description/share/naranjelio_description/meshes/BackIzq_1.stl"
+          filename="file://$(env NARANJELIO_HOME)/meshes/BackIzq_1.stl"
           scale="0.001 0.001 0.001" />
       </geometry>
@@ -548,5 +551,5 @@
       <geometry>
         <mesh
-          filename="file:///home/devuser/sinfonia/Documents/repos_varios/naranjelio_ws/install/naranjelio_description/share/naranjelio_description/meshes/BackIzq_1.stl"
+          filename="file://$(env NARANJELIO_HOME)/meshes/BackIzq_1.stl"
           scale="0.001 0.001 0.001" />
       </geometry>
@@ -563,5 +566,5 @@
       <geometry>
         <mesh
-          filename="file:///home/devuser/sinfonia/Documents/repos_varios/naranjelio_ws/install/naranjelio_description/share/naranjelio_description/meshes/BackDer_1.stl"
+          filename="file://$(env NARANJELIO_HOME)/meshes/BackDer_1.stl"
           scale="0.001 0.001 0.001" />
       </geometry>
@@ -572,5 +575,5 @@
       <geometry>
         <mesh
-          filename="file:///home/devuser/sinfonia/Documents/repos_varios/naranjelio_ws/install/naranjelio_description/share/naranjelio_description/meshes/BackDer_1.stl"
+          filename="file://$(env NARANJELIO_HOME)/meshes/BackDer_1.stl"
           scale="0.001 0.001 0.001" />
       </geometry>
@@ -587,5 +590,5 @@
       <geometry>
         <mesh
-          filename="file:///home/devuser/sinfonia/Documents/repos_varios/naranjelio_ws/install/naranjelio_description/share/naranjelio_description/meshes/FemurFrontIzq_1.stl"
+          filename="file://$(env NARANJELIO_HOME)/meshes/FemurFrontIzq_1.stl"
           scale="0.001 0.001 0.001" />
       </geometry>
@@ -596,5 +599,5 @@
       <geometry>
         <mesh
-          filename="file:///home/devuser/sinfonia/Documents/repos_varios/naranjelio_ws/install/naranjelio_description/share/naranjelio_description/meshes/FemurFrontIzq_1.stl"
+          filename="file://$(env NARANJELIO_HOME)/meshes/FemurFrontIzq_1.stl"
           scale="0.001 0.001 0.001" />
       </geometry>
@@ -611,5 +614,5 @@
       <geometry>
         <mesh
-          filename="file:///home/devuser/sinfonia/Documents/repos_varios/naranjelio_ws/install/naranjelio_description/share/naranjelio_description/meshes/FemurBackIzq_1.stl"
+          filename="file://$(env NARANJELIO_HOME)/meshes/FemurBackIzq_1.stl"
           scale="0.001 0.001 0.001" />
       </geometry>
@@ -620,5 +623,5 @@
       <geometry>
         <mesh
-          filename="file:///home/devuser/sinfonia/Documents/repos_varios/naranjelio_ws/install/naranjelio_description/share/naranjelio_description/meshes/FemurBackIzq_1.stl"
+          filename="file://$(env NARANJELIO_HOME)/meshes/FemurBackIzq_1.stl"
           scale="0.001 0.001 0.001" />
       </geometry>
@@ -635,5 +638,5 @@
       <geometry>
         <mesh
-          filename="file:///home/devuser/sinfonia/Documents/repos_varios/naranjelio_ws/install/naranjelio_description/share/naranjelio_description/meshes/FemurFrontDer_1.stl"
+          filename="file://$(env NARANJELIO_HOME)/meshes/FemurFrontDer_1.stl"
           scale="0.001 0.001 0.001" />
       </geometry>
@@ -644,5 +647,5 @@
       <geometry>
         <mesh
-          filename="file:///home/devuser/sinfonia/Documents/repos_varios/naranjelio_ws/install/naranjelio_description/share/naranjelio_description/meshes/FemurFrontDer_1.stl"
+          filename="file://$(env NARANJELIO_HOME)/meshes/FemurFrontDer_1.stl"
           scale="0.001 0.001 0.001" />
       </geometry>
@@ -659,5 +662,5 @@
       <geometry>
         <mesh
-          filename="file:///home/devuser/sinfonia/Documents/repos_varios/naranjelio_ws/install/naranjelio_description/share/naranjelio_description/meshes/FemurBackDer_1.stl"
+          filename="file://$(env NARANJELIO_HOME)/meshes/FemurBackDer_1.stl"
           scale="0.001 0.001 0.001" />
       </geometry>
@@ -668,5 +671,5 @@
       <geometry>
         <mesh
-          filename="file:///home/devuser/sinfonia/Documents/repos_varios/naranjelio_ws/install/naranjelio_description/share/naranjelio_description/meshes/FemurBackDer_1.stl"
+          filename="file://$(env NARANJELIO_HOME)/meshes/FemurBackDer_1.stl"
           scale="0.001 0.001 0.001" />
       </geometry>
@@ -683,5 +686,5 @@
       <geometry>
         <mesh
-          filename="file:///home/devuser/sinfonia/Documents/repos_varios/naranjelio_ws/install/naranjelio_description/share/naranjelio_description/meshes/TibiaLowFrontIzq_1.stl"
+          filename="file://$(env NARANJELIO_HOME)/meshes/TibiaLowFrontIzq_1.stl"
           scale="0.001 0.001 0.001" />
       </geometry>
@@ -692,5 +695,5 @@
       <geometry>
         <mesh
-          filename="file:///home/devuser/sinfonia/Documents/repos_varios/naranjelio_ws/install/naranjelio_description/share/naranjelio_description/meshes/TibiaLowFrontIzq_1.stl"
+          filename="file://$(env NARANJELIO_HOME)/meshes/TibiaLowFrontIzq_1.stl"
           scale="0.001 0.001 0.001" />
       </geometry>
@@ -707,5 +710,5 @@
       <geometry>
         <mesh
-          filename="file:///home/devuser/sinfonia/Documents/repos_varios/naranjelio_ws/install/naranjelio_description/share/naranjelio_description/meshes/TibiaLowBackIzq_1.stl"
+          filename="file://$(env NARANJELIO_HOME)/meshes/TibiaLowBackIzq_1.stl"
           scale="0.001 0.001 0.001" />
       </geometry>
@@ -716,5 +719,5 @@
       <geometry>
         <mesh
-          filename="file:///home/devuser/sinfonia/Documents/repos_varios/naranjelio_ws/install/naranjelio_description/share/naranjelio_description/meshes/TibiaLowBackIzq_1.stl"
+          filename="file://$(env NARANJELIO_HOME)/meshes/TibiaLowBackIzq_1.stl"
           scale="0.001 0.001 0.001" />
       </geometry>
@@ -731,5 +734,5 @@
       <geometry>
         <mesh
-          filename="file:///home/devuser/sinfonia/Documents/repos_varios/naranjelio_ws/install/naranjelio_description/share/naranjelio_description/meshes/TibiaLowFrontDer_1.stl"
+          filename="file://$(env NARANJELIO_HOME)/meshes/TibiaLowFrontDer_1.stl"
           scale="0.001 0.001 0.001" />
       </geometry>
@@ -740,5 +743,5 @@
       <geometry>
         <mesh
-          filename="file:///home/devuser/sinfonia/Documents/repos_varios/naranjelio_ws/install/naranjelio_description/share/naranjelio_description/meshes/TibiaLowFrontDer_1.stl"
+          filename="file://$(env NARANJELIO_HOME)/meshes/TibiaLowFrontDer_1.stl"
           scale="0.001 0.001 0.001" />
       </geometry>
@@ -755,5 +758,5 @@
       <geometry>
         <mesh
-          filename="file:///home/devuser/sinfonia/Documents/repos_varios/naranjelio_ws/install/naranjelio_description/share/naranjelio_description/meshes/TibiaLowBackDer_1.stl"
+          filename="file://$(env NARANJELIO_HOME)/meshes/TibiaLowBackDer_1.stl"
           scale="0.001 0.001 0.001" />
       </geometry>
@@ -764,5 +767,5 @@
       <geometry>
         <mesh
-          filename="file:///home/devuser/sinfonia/Documents/repos_varios/naranjelio_ws/install/naranjelio_description/share/naranjelio_description/meshes/TibiaLowBackDer_1.stl"
+          filename="file://$(env NARANJELIO_HOME)/meshes/TibiaLowBackDer_1.stl"
           scale="0.001 0.001 0.001" />
       </geometry>
@@ -779,5 +782,5 @@
       <geometry>
         <mesh
-          filename="file:///home/devuser/sinfonia/Documents/repos_varios/naranjelio_ws/install/naranjelio_description/share/naranjelio_description/meshes/TibiaHighFrontIzq_1.stl"
+          filename="file://$(env NARANJELIO_HOME)/meshes/TibiaHighFrontIzq_1.stl"
           scale="0.001 0.001 0.001" />
       </geometry>
@@ -788,5 +791,5 @@
       <geometry>
         <mesh
-          filename="file:///home/devuser/sinfonia/Documents/repos_varios/naranjelio_ws/install/naranjelio_description/share/naranjelio_description/meshes/TibiaHighFrontIzq_1.stl"
+          filename="file://$(env NARANJELIO_HOME)/meshes/TibiaHighFrontIzq_1.stl"
           scale="0.001 0.001 0.001" />
       </geometry>
@@ -797,5 +800,5 @@
       <origin rpy="0 0 0" xyz="0.0016921596049667281 -0.015756854381915097 0.002778854381984844" />
       <mass value="0.0007780427273559296" />
-      <inertia ixx="0.0" ixy="0.0" ixz="-0.0" iyy="0.0" iyz="0.0" izz="0.0" />
+      <inertia ixx="1e-06" ixy="0.0" ixz="0.0" iyy="1e-06" iyz="0.0" izz="1e-06" />
     </inertial>
     <visual>
@@ -803,5 +806,5 @@
       <geometry>
         <mesh
-          filename="file:///home/devuser/sinfonia/Documents/repos_varios/naranjelio_ws/install/naranjelio_description/share/naranjelio_description/meshes/PivotTibiaFrontIzq_1.stl"
+          filename="file://$(env NARANJELIO_HOME)/meshes/PivotTibiaFrontIzq_1.stl"
           scale="0.001 0.001 0.001" />
       </geometry>
@@ -812,5 +815,5 @@
       <geometry>
         <mesh
-          filename="file:///home/devuser/sinfonia/Documents/repos_varios/naranjelio_ws/install/naranjelio_description/share/naranjelio_description/meshes/PivotTibiaFrontIzq_1.stl"
+          filename="file://$(env NARANJELIO_HOME)/meshes/PivotTibiaFrontIzq_1.stl"
           scale="0.001 0.001 0.001" />
       </geometry>
@@ -821,5 +824,5 @@
       <origin rpy="0 0 0" xyz="0.0016921596049660897 0.01570761399426379 0.0027701719731016983" />
       <mass value="0.0007780427273559296" />
-      <inertia ixx="0.0" ixy="-0.0" ixz="-0.0" iyy="0.0" iyz="-0.0" izz="0.0" />
+      <inertia ixx="1e-06" ixy="0.0" ixz="0.0" iyy="1e-06" iyz="0.0" izz="1e-06" />
     </inertial>
     <visual>
@@ -827,5 +830,5 @@
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